Commit message: Updated camera position from bottom to top of the chassis.
This is the bug fix after project review. Initially this problem was hidden because of two models of robot existing with the same name. After removing one instance of the robot inside world instance this problem become visible,

File: my_robot/urdf/my_robot.xacro (robot description, xacro)
@@ -11,5 +11,5 @@
     <origin xyz="0 0 0" rpy="0 0 0"/>
     <child link="left_wheel"/>
-    <parent link="chassis"/>
+    <parent link="robot_footprint"/>
     <axis xyz="0 1 0" rpy="0 0 0"/>
     <limit effort="10000" velocity="1000"/>
@@ -19,5 +19,5 @@
     <origin xyz="0 0 0" rpy="0 0 0"/>
     <child link="right_wheel"/>
-    <parent link="chassis"/>
+    <parent link="robot_footprint"/>
     <axis xyz="0 1 0" rpy="0 0 0"/>
     <limit effort="10000" velocity="1000"/>
@@ -33,5 +33,5 @@
   </joint>
   <joint type="fixed" name="hokuyo_joint">
-    <origin xyz="0 0 0" rpy="0 0 0"/>
+    <origin xyz="0 0 0.2" rpy="0 0 0"/>
     <child link="hokuyo"/>
     <parent link="chassis"/>
